File: door_if2/door_if2.kicad_pcb (KiCad board)
At the start: 2 copper layers, 74 parts, among them J1 Conn_01x08, J2 Raspberry_Pi_2_3, J3 Conn_02x05_Odd_Even, J4 Conn_01x08, J5 Conn_02x05_Odd_Even, Q1 IRF7389, Q2 IRF7389, Q3 IRF7389, Q4 IRF7389, U1 LTV-247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

Commit message: added boards
Parts:
- added R30: 10k, Resistor_SMD:R_0603_1608Metric_Pad1.05x0.95mm_HandSolder, F.Cu at (133.9, 72.7)
- added R31: 10k, Resistor_SMD:R_0603_1608Metric_Pad1.05x0.95mm_HandSolder, F.Cu at (133.9, 75.6)
- added R32: 10k, Resistor_SMD:R_0603_1608Metric_Pad1.05x0.95mm_HandSolder, F.Cu at (133.9, 78.1)
- added R33: 10k, Resistor_SMD:R_0603_1608Metric_Pad1.05x0.95mm_HandSolder, F.Cu at (130.5, 84.0)
- Q1, Q2, Q3, Q4: value IRF7389 -> IRF7343
- R21, R22: moved to B.Cu
- moved R20 36.7 mm to (102.1, 70.3)
- moved R21 35.7 mm to (101.9, 72.6)
- moved R22 15.4 mm to (122.0, 78.9), turned to 270 degrees
- moved R1 6.80 mm to (107.3, 82.8), turned to 270 degrees
- moved R19 3.81 mm to (129.4, 70.5), turned to 180 degrees
- moved R3 3.05 mm to (104.1, 82.8), turned to 270 degrees
- moved R2 1.14 mm to (105.7, 82.8), turned to 270 degrees
- moved R5 1.02 mm to (102.5, 82.8)
Connections:
- JP1 pad 1: Net-(JP1-Pad1) -> +12V
- JP1 pad 2: +12V -> Net-(JP1-Pad2)
- JP10 pad 1: Net-(JP10-Pad1) -> GNDA
- JP10 pad 2: GNDA -> Net-(JP10-Pad2)
- JP11 pad 1: Net-(JP11-Pad1) -> +12V
- JP11 pad 2: +12V -> Net-(JP11-Pad2)
- JP12 pad 1: Net-(JP12-Pad1) -> GNDA
- JP12 pad 2: GNDA -> Net-(JP12-Pad2)
- JP13 pad 1: Net-(JP13-Pad1) -> +12V
- JP13 pad 2: +12V -> Net-(JP13-Pad2)
- JP14 pad 1: Net-(JP14-Pad1) -> GNDA
- JP14 pad 2: GNDA -> Net-(JP14-Pad2)
- JP15 pad 1: Net-(JP15-Pad1) -> +12V
- JP15 pad 2: +12V -> Net-(JP15-Pad2)
- JP16 pad 1: Net-(JP16-Pad1) -> GNDA
- JP16 pad 2: GNDA -> Net-(JP16-Pad2)
- JP2 pad 1: Net-(JP2-Pad1) -> GNDA
- JP2 pad 2: GNDA -> Net-(JP2-Pad2)
- JP3 pad 1: Net-(JP3-Pad1) -> +12V
- JP3 pad 2: +12V -> Net-(JP3-Pad2)
- JP4 pad 1: Net-(JP4-Pad1) -> GNDA
- JP4 pad 2: GNDA -> Net-(JP4-Pad2)
- JP5 pad 1: Net-(JP5-Pad1) -> +12V
- JP5 pad 2: +12V -> Net-(JP5-Pad2)
- JP6 pad 1: Net-(JP6-Pad1) -> GNDA
- JP6 pad 2: GNDA -> Net-(JP6-Pad2)
- JP7 pad 1: Net-(JP7-Pad1) -> +12V
- JP7 pad 2: +12V -> Net-(JP7-Pad2)
- JP8 pad 1: Net-(JP8-Pad1) -> GNDA
- JP8 pad 2: GNDA -> Net-(JP8-Pad2)
- JP9 pad 1: Net-(JP9-Pad1) -> +12V
- JP9 pad 2: +12V -> Net-(JP9-Pad2)
- R10 pad 2: Net-(JP1-Pad1) -> Net-(JP1-Pad2)
- R11 pad 2: Net-(JP3-Pad1) -> Net-(JP3-Pad2)
- R12 pad 2: Net-(JP5-Pad1) -> Net-(JP5-Pad2)
- R14 pad 2: Net-(JP7-Pad1) -> Net-(JP7-Pad2)
- R15 pad 2: Net-(JP9-Pad1) -> Net-(JP9-Pad2)
- R16 pad 2: Net-(JP11-Pad1) -> Net-(JP11-Pad2)
- R17 pad 2: Net-(JP13-Pad1) -> Net-(JP13-Pad2)
- R18 pad 2: Net-(JP15-Pad1) -> Net-(JP15-Pad2)
- U1 pad 2: Net-(JP2-Pad1) -> Net-(JP2-Pad2)
- U1 pad 4: Net-(JP4-Pad1) -> Net-(JP4-Pad2)
- U1 pad 6: Net-(JP6-Pad1) -> Net-(JP6-Pad2)
- U1 pad 8: Net-(JP8-Pad1) -> Net-(JP8-Pad2)
- U2 pad 2: Net-(JP10-Pad1) -> Net-(JP10-Pad2)
- U2 pad 4: Net-(JP12-Pad1) -> Net-(JP12-Pad2)
- U2 pad 6: Net-(JP14-Pad1) -> Net-(JP14-Pad2)
- U2 pad 8: Net-(JP16-Pad1) -> Net-(JP16-Pad2)
- U3 pad 10: Net-(JP23-Pad2) -> Net-(R33-Pad1)
- U3 pad 12: Net-(JP21-Pad2) -> Net-(R32-Pad1)
- U3 pad 14: Net-(JP19-Pad2) -> Net-(R31-Pad1)
- U3 pad 16: Net-(JP17-Pad2) -> Net-(R30-Pad1)
Routing:
- net +12V: track 150.4 -> 290.1 mm, vias 2 -> 10
- net S_IN7: track 0.00 -> 96.0 mm, vias 0 -> 2
- net +3V3: track 0.00 -> 87.1 mm, vias 0 -> 15
- net Net-(JP16-Pad2): track 0.00 -> 78.0 mm, vias 0 -> 1
- net Net-(JP16-Pad1): track 76.1 -> 0.00 mm, vias 1 -> 0
- net Net-(JP14-Pad1): track 72.2 -> 0.00 mm, vias 1 -> 0
- net Net-(JP14-Pad2): track 0.00 -> 72.0 mm, vias 0 -> 1
- net S_IN6: track 0.00 -> 65.6 mm, vias 0 -> 2
- net S_IN2: track 0.00 -> 63.5 mm, vias 0 -> 1
- net Net-(JP15-Pad2): track 0.00 -> 62.6 mm, vias 0 -> 1
- net S_IN8: track 0.00 -> 60.1 mm, vias 0 -> 2
- net Net-(JP15-Pad1): track 59.4 -> 0.00 mm, vias 1 -> 0
- net Net-(JP13-Pad2): track 0.00 -> 56.0 mm, vias 0 -> 1
- net S_IN5: track 0.00 -> 54.6 mm, vias 0 -> 2
- net Net-(JP13-Pad1): track 52.9 -> 0.00 mm, vias 1 -> 0
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- added copper zone on B.Cu, net GND
Other:
- board outline added: 65 x 56.5 mm
- board text added: "ZAM door_if2 20220304 ChrisC"
