File: door_if2/door_if2.sch (KiCad schematic (older format))
At the start: 74 parts, among them J1 Conn_01x08, J2 Raspberry_Pi_2_3, J3 Conn_02x05_Odd_Even, J4 Conn_01x08, J5 Conn_02x05_Odd_Even, Q1 IRF7389, Q2 IRF7389, Q3 IRF7389, Q4 IRF7389, U1 LTV-247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

Commit message: added boards
Parts:
- added R30, R31, R32, R33: 10k, Resistor_SMD:R_0603_1608Metric_Pad1.05x0.95mm_HandSolder, symbol Device:R
- Q1, Q2, Q3, Q4: value IRF7389 -> IRF7343
Connections:
- net +12V: now also JP1.1 (A), JP11.1 (A), JP13.1 (A), JP15.1 (A), JP3.1 (A), JP5.1 (A), JP7.1 (A), JP9.1 (A); no longer JP1.2 (C), JP11.2 (C), JP13.2 (C), JP15.2 (C), JP3.2 (C), JP5.2 (C), JP7.2 (C), JP9.2 (C)
- net GNDA: now also JP10.1 (A), JP12.1 (A), JP14.1 (A), JP16.1 (A), JP2.1 (A), JP4.1 (A), JP6.1 (A), JP8.1 (A); no longer JP10.2 (C), JP12.2 (C), JP14.2 (C), JP16.2 (C), JP2.2 (C), JP4.2 (C), JP6.2 (C), JP8.2 (C)
- net at U3.16: now also R30.1; no longer JP17.2 (C)
- net at U3.14: now also R31.1; no longer JP19.2 (C)
- net at U3.12: now also R32.1; no longer JP21.2 (C)
- net at U3.10: now also R33.1; no longer JP23.2 (C)
- net at U1.2: now also JP2.2 (C); no longer JP2.1 (A)
- net at R10.2: now also JP1.2 (C); no longer JP1.1 (A)
- net at U1.4: now also JP4.2 (C); no longer JP4.1 (A)
- net at R11.2: now also JP3.2 (C); no longer JP3.1 (A)
- net at U1.6: now also JP6.2 (C); no longer JP6.1 (A)
- net at R12.2: now also JP5.2 (C); no longer JP5.1 (A)
- net at U1.8: now also JP8.2 (C); no longer JP8.1 (A)
- net at R14.2: now also JP7.2 (C); no longer JP7.1 (A)
- net at U2.2: now also JP10.2 (C); no longer JP10.1 (A)
- net at R15.2: now also JP9.2 (C); no longer JP9.1 (A)
- net at U2.4: now also JP12.2 (C); no longer JP12.1 (A)
- net at R16.2: now also JP11.2 (C); no longer JP11.1 (A)
- net at U2.6: now also JP14.2 (C); no longer JP14.1 (A)
- net at R17.2: now also JP13.2 (C); no longer JP13.1 (A)
- net at U2.8: now also JP16.2 (C); no longer JP16.1 (A)
- net at R18.2: now also JP15.2 (C); no longer JP15.1 (A)
- new net: JP17.2 (C), R30.2
- new net: JP19.2 (C), R31.2
- new net: JP21.2 (C), R32.2
- new net: JP23.2 (C), R33.2
Other:
- moved on the sheet: R19, R20, R21, R22, U3A, U3B, U3C, U3D
