File: pcb/door_if4_usb/door_if4_usb.kicad_sch (KiCad schematic)
At the start: 12 parts, among them J1 WAGO 250-206, J2 WAGO 250-206, J3 WAGO 250-206, U1 Pico

Commit message: almost completed door_if4_usb for manufacturing
Parts:
- removed H4: MountingHole, MountingHole:MountingHole_3.2mm_M3_DIN965, symbol Mechanical:MountingHole
Changed lines of the file:
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@@
-    )
-  )
-  (symbol (lib_id "Mechanical:MountingHole") (at 133.35 177.8 0) (unit 1)
-    (in_bom yes) (on_board yes) (dnp no) (fields_autoplaced)
-    (property "Reference" "H4" (at 135.89 177.165 0)
-      (effects (font (size 1.27 1.27)) (justify left))
-    )
-    (property "Value" "MountingHole" (at 135.89 179.705 0)
-      (effects (font (size 1.27 1.27)) (justify left))
-    )
-    (property "Footprint" "MountingHole:MountingHole_3.2mm_M3_DIN965" (at 133.35 177.8 0)
-      (effects (font (size 1.27 1.27)) hide)
-    )
-    (property "Datasheet" "~" (at 133.35 177.8 0)
-      (effects (font (size 1.27 1.27)) hide)
-    )
-    (instances
-      (project "door_if4_usb"
-        (path "/c43b7d50-4f10-4f9a-abda-bb9ac9eb6c0d"
-          (reference "H4") (unit 1)
-        )
-      )
     )
   )

Commit message: added final if4 design
Parts:
- C1, C2: footprint Capacitor_SMD:C_0402_1005Metric -> Capacitor_SMD:C_0805_2012Metric
Changed lines of the file:
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@@
       (effects (font (size 1.27 1.27)) (justify left))
     )
-    (property "Footprint" "Capacitor_SMD:C_0402_1005Metric" (at 58.1152 158.75 0)
+    (property "Footprint" "Capacitor_SMD:C_0805_2012Metric" (at 58.1152 158.75 0)
       (effects (font (size 1.27 1.27)) hide)
     )
@@
       (effects (font (size 1.27 1.27)) (justify left))
     )
-    (property "Footprint" "Capacitor_SMD:C_0402_1005Metric" (at 33.3502 159.385 0)
+    (property "Footprint" "Capacitor_SMD:C_0805_2012Metric" (at 33.3502 159.385 0)
       (effects (font (size 1.27 1.27)) hide)
     )
