File: pcb/door_if4_usb/door_if4_usb_inch2.kicad_sch (KiCad schematic)
At the start: 9 parts, among them U2 LTV-247

Commit message: almost completed door_if4_usb for manufacturing
Connections:
- net GND: now reaches U2.11, U2.13, U2.15, U2.9
Changed lines of the file:
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@@
   (junction (at 151.765 102.87) (diameter 0) (color 0 0 0 0)
   )
+  (junction (at 130.81 118.11) (diameter 0) (color 0 0 0 0)
+  )
   (junction (at 153.67 110.49) (diameter 0) (color 0 0 0 0)
   )
@@
     (stroke (width 0) (type default))
   )
-  (wire (pts (xy 130.175 118.11) (xy 133.35 118.11))
+  (wire (pts (xy 130.175 118.11) (xy 130.81 118.11))
     (stroke (width 0) (type default))
   )
@@
     (stroke (width 0) (type default))
   )
+  (wire (pts (xy 130.81 118.11) (xy 130.81 121.92))
+    (stroke (width 0) (type default))
+  )
   (wire (pts (xy 113.665 110.49) (xy 113.665 100.33))
     (stroke (width 0) (type default))
@@
   )
   (wire (pts (xy 111.76 83.185) (xy 125.095 83.185))
+    (stroke (width 0) (type default))
+  )
+  (wire (pts (xy 130.81 118.11) (xy 133.35 118.11))
     (stroke (width 0) (type default))
   )
@@
         )
       )
+    )
+  )
+  (symbol (lib_id "power:GND") (at 130.81 121.92 0) (unit 1)
+    (in_bom yes) (on_board yes) (dnp no) (fields_autoplaced)
+    (property "Reference" "#PWR074" (at 130.81 128.27 0)
+      (effects (font (size 1.27 1.27)) hide)
+    )
+    (property "Value" "GND" (at 130.81 127 0)
+      (effects (font (size 1.27 1.27)))
+    )
+    (property "Footprint" "" (at 130.81 121.92 0)
+      (effects (font (size 1.27 1.27)) hide)
+    )
+    (property "Datasheet" "" (at 130.81 121.92 0)
+      (effects (font (size 1.27 1.27)) hide)
+    )
+    (pin "1")
+    (instances
+      (project "door_if4_usb"
+        (path "/c43b7d50-4f10-4f9a-abda-bb9ac9eb6c0d/4f518f41-fe71-4a68-a821-742113f3b8ca"
+          (reference "#PWR074") (unit 1)
+        )
+        (path "/c43b7d50-4f10-4f9a-abda-bb9ac9eb6c0d/2cbe48b6-fef4-4f3d-887a-472992e5d1b2"
+          (reference "#PWR075") (unit 1)
+        )
+        (path "/c43b7d50-4f10-4f9a-abda-bb9ac9eb6c0d/73c95cf2-9040-41a4-83f4-e10df379f760"
+          (reference "#PWR076") (unit 1)
+        )
+        (path "/c43b7d50-4f10-4f9a-abda-bb9ac9eb6c0d/11577c63-84b8-4065-a797-984cf6a4b692"
+          (reference "#PWR077") (unit 1)
+        )
+      )

Commit message: added final if4 design
Parts:
- added D26, D30, D34, D38: D, Diode_SMD:D_SOD-523, symbol Device:D
- R18, R19, R20, R21: value 22k -> 10k
Connections:
- net I_IN1: now also D26.2 (A); no longer U2.1
- net I_IN2: now also D34.2 (A); no longer U2.5
- net at R20.1, R21.1, U2.6: now also D38.2 (A); no longer U2.7
- net at R18.1, R19.1, U2.2: now also D30.2 (A); no longer U2.3
- new net: D38.1 (K), U2.7
- new net: D30.1 (K), U2.3
- new net: D34.1 (K), U2.5
- new net: D26.1 (K), U2.1
Other:
- moved on the sheet: R18, R19, R20, R21
